File: hardware/pcb_kicad/pcb_kicad_routed.kicad_pcb (KiCad board)
At the start: 2 copper layers, 105.4 x 41.9 mm, 26 parts, among them J1 Barrel_Jack, J2 Screw_Terminal_01x02, J3 Screw_Terminal_01x02, J4 Screw_Terminal_01x02, J5 Screw_Terminal_01x02, J6 Conn_02x05_Top_Bottom, Q1 IRLB8721PBF, Q2 IRLB8721PBF, U1 LM7805_TO220

Commit message: best run so far
Parts:
- added J7: Conn_01x05_Male, Connector_PinHeader_2.54mm:PinHeader_1x05_P2.54mm_Vertical, F.Cu at (100.3, 92.7)
- J6: value Conn_02x05_Top_Bottom -> Conn_01x06_Male; footprint Connector_IDC:IDC-Header_2x05_P2.54mm_Vertical -> Connector_PinHeader_2.54mm:PinHeader_1x06_P2.54mm_Vertical
- moved C1 23.0 mm to (113.0, 86.4)
- moved H1 21.6 mm to (63.5, 64.8)
- moved H2 21.6 mm to (63.5, 96.5)
- moved J6 20.4 mm to (85.1, 67.3), turned to 270 degrees
- moved U1 19.4 mm to (111.8, 78.7), turned to 90 degrees
- moved JP2 14.0 mm to (132.1, 80.0)
- moved Driver1 10.2 mm to (118.1, 86.4)
- moved JP3 10.2 mm to (124.5, 80.0)
- moved RV1 8.89 mm to (72.4, 97.8)
- moved JP1 6.35 mm to (128.3, 80.0)
- moved RV2 6.27 mm to (111.8, 97.8)
- moved J4 1.27 mm to (148.6, 64.8)
- moved J3 1.27 mm to (127.0, 64.8)
- moved RV3 1.11 mm to (146.2, 97.8)
Connections:
- Nano1 pad 10: Net-(J6-Pad1) -> GND
- Nano1 pad 11: Net-(J6-Pad2) -> Net-(J6-Pad1)
- Nano1 pad 12: Net-(J6-Pad3) -> Net-(J6-Pad2)
- Nano1 pad 13: Net-(J6-Pad4) -> Net-(J6-Pad3)
- Nano1 pad 14: (no net) -> Net-(J6-Pad4)
- Nano1 pad 15: (no net) -> Net-(J6-Pad5)
- Nano1 pad 16: (no net) -> Net-(J6-Pad6)
- Nano1 pad 22: Net-(J6-Pad5) -> Net-(J7-Pad5)
- Nano1 pad 23: Net-(J6-Pad6) -> Net-(J7-Pad4)
- Nano1 pad 24: Net-(J6-Pad7) -> Net-(J7-Pad3)
- Nano1 pad 25: Net-(J6-Pad8) -> Net-(J7-Pad2)
- Nano1 pad 26: (no net) -> Net-(J7-Pad1)
Routing:
- net +5V: track 200.1 -> 144.5 mm, vias 1 -> 0
- net Net-(J6-Pad8): track 34.7 -> 0.00 mm
- net Net-(J6-Pad7): track 27.7 -> 0.00 mm
- net Net-(J6-Pad6): track 45.3 -> 23.0 mm
- net Net-(J6-Pad5): track 26.3 -> 11.0 mm
- net Net-(J6-Pad3): track 23.3 -> 11.0 mm
- net Net-(Driver1-Pad16): track 17.0 -> 28.3 mm
- net Net-(J7-Pad5): track 0.00 -> 11.0 mm
- net Net-(J7-Pad3): track 0.00 -> 11.0 mm
- net Net-(J7-Pad2): track 0.00 -> 11.0 mm
- net Net-(J7-Pad1): track 0.00 -> 11.0 mm
- net Net-(J7-Pad4): track 0.00 -> 11.0 mm
- net Net-(Driver1-Pad15): track 23.2 -> 34.0 mm
- net Net-(Driver1-Pad9): track 41.7 -> 52.3 mm
- net Net-(J6-Pad4): track 19.8 -> 11.0 mm
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Other:
- net class Power: trace_width 0.7 -> 1
- board text added: "+12v"
- board text removed: "+"
- board text removed: "+12V"
- board text removed: "1A"
- board text removed: "1B"
- board text removed: "2A"
- board text removed: "2B"
- board text removed: "<- USB"
- board text removed: "Ext"
- board text removed: "Flash"
- board text removed: "Frames"
- board text removed: "Leds"
- board text removed: "Power"
- board text removed: "Speed"
- board text removed: "Stepper"
- board text removed: "ZOETROPE V1"
