File: hardware/pcb_kicad/pcb_kicad.kicad_pcb (KiCad board)
At the start: 2 copper layers, 101.6 x 44.5 mm, 17 parts, among them J1 Barrel_Jack, J2 Screw_Terminal_01x04, J3 Screw_Terminal_01x06, Q1 IRLB8721PBF, Q2 IRLB8721PBF, Q3 IRLB8721PBF

Commit message: better latyout?
Parts:
- added J4: Screw_Terminal_01x02, TerminalBlock:TerminalBlock_bornier-2_P5.08mm, F.Cu at (162.6, 64.8)
- added J5: Screw_Terminal_01x02, TerminalBlock:TerminalBlock_bornier-2_P5.08mm, F.Cu at (127.0, 64.8)
- added J6: Screw_Terminal_01x02, TerminalBlock:TerminalBlock_bornier-2_P5.08mm, F.Cu at (151.1, 64.8)
- J2: value Screw_Terminal_01x04 -> Screw_Terminal_01x02; footprint TerminalBlock:TerminalBlock_bornier-4_P5.08mm -> TerminalBlock:TerminalBlock_bornier-2_P5.08mm
- J3: value Screw_Terminal_01x06 -> Screw_Terminal_01x02; footprint TerminalBlock:TerminalBlock_bornier-6_P5.08mm -> TerminalBlock:TerminalBlock_bornier-2_P5.08mm
- moved Q3 53.5 mm to (146.1, 74.9)
- moved J3 49.3 mm to (138.4, 64.8), turned to 180 degrees
- moved J2 36.4 mm to (174.0, 64.8), turned to 180 degrees
- moved R1 36.1 mm to (146.1, 88.9), turned to 90 degrees
- moved J1 34.4 mm to (193.0, 72.4)
- moved R3 32.0 mm to (157.5, 78.7), turned to 270 degrees
- moved Q2 31.1 mm to (157.5, 74.9)
- moved RV3 30.5 mm to (166.4, 97.8)
- moved R2 29.6 mm to (151.1, 88.9), turned to 90 degrees
- moved R5 19.9 mm to (168.9, 78.7), turned to 270 degrees
- moved Q1 19.1 mm to (168.9, 74.9)
- moved RV2 14.1 mm to (119.5, 97.8)
- moved R4 11.9 mm to (162.6, 78.7), turned to 270 degrees
- moved R6 11.9 mm to (174.0, 88.9), turned to 90 degrees
- moved Nano1 7.41 mm to (110.5, 71.1)
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Connections:
- J3 pad 1: Net-(J3-Pad1) -> Net-(Driver1-Pad5)
- J3 pad 2: +12V -> Net-(Driver1-Pad6)
- Q1 pad 2: Net-(J3-Pad1) -> Net-(J4-Pad1)
- Q2 pad 2: Net-(J3-Pad3) -> Net-(J5-Pad1)
- Q3 pad 2: Net-(J3-Pad5) -> Net-(J6-Pad1)
Routing:
- net +12V: track 46.6 -> 134.9 mm
- net Net-(Nano1-Pad8): track 0.00 -> 56.7 mm
- net Net-(J5-Pad1): track 0.00 -> 37.2 mm
- net Net-(Q3-Pad1): track 0.00 -> 36.7 mm
- net Net-(Nano1-Pad21): track 56.8 -> 88.6 mm
- net Net-(Q1-Pad1): track 0.00 -> 28.9 mm
- net Net-(Driver1-Pad3): track 37.6 -> 66.3 mm
- net GND: track 190.7 -> 217.7 mm
- net Net-(Driver1-Pad4): track 33.0 -> 56.4 mm
- net Net-(Nano1-Pad20): track 28.9 -> 44.3 mm
- net Net-(J4-Pad1): track 0.00 -> 14.2 mm
- net +5V: track 106.6 -> 118.4 mm
- net Net-(J6-Pad1): track 0.00 -> 11.2 mm
- net Net-(Q2-Pad1): track 0.00 -> 8.89 mm
- net Net-(Nano1-Pad19): track 21.5 -> 13.6 mm
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Other:
- board size 101.6 x 44.5 mm -> 132.1 x 41.9 mm
- net class Default: trace_width 0.25 -> 0.5
- net class Power added: clearance 0.2, trace_width 1, via_dia 0.8, via_drill 0.4

Commit message: rework
Parts:
- removed Q3: IRLB8721PBF, Package_TO_SOT_THT:TO-220-3_Vertical
- removed R5: 220, Resistor_THT:R_Axial_DIN0207_L6.3mm_D2.5mm_P10.16mm_Horizontal
- removed R6: 100K, Resistor_THT:R_Axial_DIN0207_L6.3mm_D2.5mm_P10.16mm_Horizontal
- added C1: 100uF, Capacitor_THT:CP_Radial_D6.3mm_P2.50mm, F.Cu at (137.2, 78.7)
- added H1: MountingHole, MountingHole:MountingHole_3.2mm_M3, F.Cu at (63.5, 64.8)
- added H2: MountingHole, MountingHole:MountingHole_3.2mm_M3, F.Cu at (63.5, 96.5)
- added H3: MountingHole, MountingHole:MountingHole_3.2mm_M3, F.Cu at (135.9, 64.8)
- added H4: MountingHole, MountingHole:MountingHole_3.2mm_M3, F.Cu at (135.9, 96.5)
- added J7: Conn_01x05_Male, Connector_PinHeader_2.54mm:PinHeader_1x05_P2.54mm_Vertical, F.Cu at (100.3, 92.7)
- added JP1: SolderJumper_3_Bridged12, Jumper:SolderJumper-3_P1.3mm_Bridged12_Pad1.0x1.5mm_NumberLabels, F.Cu at (119.4, 78.8)
- added JP2: SolderJumper_3_Bridged12, Jumper:SolderJumper-3_P1.3mm_Bridged12_Pad1.0x1.5mm_NumberLabels, F.Cu at (123.2, 78.8)
- added JP3: SolderJumper_3_Bridged12, Jumper:SolderJumper-3_P1.3mm_Bridged12_Pad1.0x1.5mm_NumberLabels, F.Cu at (115.6, 78.7)
- J6: value Screw_Terminal_01x02 -> Conn_01x06_Male; footprint TerminalBlock:TerminalBlock_bornier-2_P5.08mm -> Connector_PinHeader_2.54mm:PinHeader_1x06_P2.54mm_Vertical
- moved J1 93.0 mm to (100.3, 64.8), turned to 180 degrees
- moved J6 66.1 mm to (85.1, 67.3), turned to 270 degrees
- moved J2 58.4 mm to (115.6, 64.8)
- moved J5 33.0 mm to (160.0, 64.8)
- moved Q1 25.4 mm to (143.5, 74.9)
- moved RV3 20.2 mm to (146.2, 97.8)
- moved J4 14.0 mm to (148.6, 64.8)
- moved Driver1 11.5 mm to (109.2, 85.1)
- moved J3 11.4 mm to (127.0, 64.8)
- moved Nano1 8.98 mm to (101.6, 72.4)
- moved RV2 7.70 mm to (111.8, 97.8)
- moved R1 2.54 mm to (143.5, 88.9)
- moved Q2 2.54 mm to (154.9, 74.9)
- moved R2 2.54 mm to (148.6, 88.9)
- moved R3 2.54 mm to (154.9, 78.7)
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Connections:
- Driver1 pad 10: (no net) -> Net-(Driver1-Pad10)
- Driver1 pad 11: (no net) -> Net-(Driver1-Pad11)
- Driver1 pad 12: (no net) -> Net-(Driver1-Pad12)
- J2 pad 1: Net-(Driver1-Pad3) -> Net-(Driver1-Pad4)
- J2 pad 2: Net-(Driver1-Pad4) -> Net-(Driver1-Pad3)
- J3 pad 1: Net-(Driver1-Pad5) -> Net-(Driver1-Pad6)
- J3 pad 2: Net-(Driver1-Pad6) -> Net-(Driver1-Pad5)
- J6 pad 2: +12V -> Net-(J6-Pad2)
- Nano1 pad 11: (no net) -> Net-(J6-Pad1)
- Nano1 pad 12: (no net) -> Net-(J6-Pad2)
- Nano1 pad 13: (no net) -> Net-(J6-Pad3)
- Nano1 pad 14: (no net) -> Net-(J6-Pad4)
- Nano1 pad 15: (no net) -> Net-(J6-Pad5)
- Nano1 pad 16: (no net) -> Net-(J6-Pad6)
- Nano1 pad 22: (no net) -> Net-(J7-Pad5)
- Nano1 pad 23: (no net) -> Net-(J7-Pad4)
- Nano1 pad 24: (no net) -> Net-(J7-Pad3)
- Nano1 pad 25: (no net) -> Net-(J7-Pad2)
- Nano1 pad 26: (no net) -> Net-(J7-Pad1)
Routing:
- net GND: track 217.7 -> 0.00 mm
- net +12V: track 134.9 -> 0.00 mm
- net +5V: track 118.4 -> 0.00 mm
- net Net-(Nano1-Pad21): track 88.6 -> 0.00 mm
- net Net-(Driver1-Pad3): track 66.3 -> 0.00 mm
- net Net-(Nano1-Pad8): track 56.7 -> 0.00 mm
- net Net-(Driver1-Pad4): track 56.4 -> 0.00 mm
- net Net-(Driver1-Pad9): track 45.2 -> 0.00 mm
- net Net-(Nano1-Pad20): track 44.3 -> 0.00 mm
- net Net-(J5-Pad1): track 37.2 -> 0.00 mm
- net Net-(Q3-Pad1): track 36.7 -> 0.00 mm
- net Net-(Driver1-Pad6): track 31.3 -> 0.00 mm
- net Net-(Q1-Pad1): track 28.9 -> 0.00 mm
- net Net-(Driver1-Pad15): track 27.0 -> 0.00 mm
- net Net-(Driver1-Pad5): track 22.2 -> 0.00 mm
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Other:
- board size 132.1 x 41.9 mm -> 105.4 x 41.9 mm
- board text added: "+12v"
- board text added: "GND"
- board text added: "Stepper"

Commit message: best run so far
Parts:
- removed J7: Conn_01x05_Male, Connector_PinHeader_2.54mm:PinHeader_1x05_P2.54mm_Vertical
- added U1: LM7805_TO220, Package_TO_SOT_THT:TO-220-3_Vertical, F.Cu at (130.8, 74.9)
- J6: value Conn_01x06_Male -> Conn_02x05_Top_Bottom; footprint Connector_PinHeader_2.54mm:PinHeader_1x06_P2.54mm_Vertical -> Connector_IDC:IDC-Header_2x05_P2.54mm_Vertical
- moved H1 21.6 mm to (85.1, 64.8)
- moved H2 21.6 mm to (85.1, 96.5)
- moved J6 20.4 mm to (64.8, 66.0), turned to 90 degrees
- moved RV1 8.89 mm to (63.5, 97.8)
- moved RV2 6.27 mm to (105.6, 97.8)
- moved C1 5.24 mm to (135.9, 83.8)
- moved JP2 5.23 mm to (118.1, 80.0)
- moved JP1 2.83 mm to (121.9, 80.0)
- moved JP3 1.80 mm to (114.3, 80.0)
- moved Driver1 1.80 mm to (108.0, 86.4)
- moved J4 1.27 mm to (149.9, 64.8)
- moved J3 1.27 mm to (125.7, 64.8)
- moved RV3 1.11 mm to (147.3, 97.8)
Connections:
- Nano1 pad 10: GND -> Net-(J6-Pad1)
- Nano1 pad 11: Net-(J6-Pad1) -> Net-(J6-Pad2)
- Nano1 pad 12: Net-(J6-Pad2) -> Net-(J6-Pad3)
- Nano1 pad 13: Net-(J6-Pad3) -> Net-(J6-Pad4)
- Nano1 pad 14: Net-(J6-Pad4) -> (no net)
- Nano1 pad 15: Net-(J6-Pad5) -> (no net)
- Nano1 pad 16: Net-(J6-Pad6) -> (no net)
- Nano1 pad 22: Net-(J7-Pad5) -> Net-(J6-Pad5)
- Nano1 pad 23: Net-(J7-Pad4) -> Net-(J6-Pad6)
- Nano1 pad 24: Net-(J7-Pad3) -> Net-(J6-Pad7)
- Nano1 pad 25: Net-(J7-Pad2) -> Net-(J6-Pad8)
- Nano1 pad 26: Net-(J7-Pad1) -> (no net)
- Nano1 pad 30: +12V -> (no net)
Routing:
- net GND: track 0.00 -> 226.7 mm
- net +5V: track 0.00 -> 200.1 mm, vias 0 -> 1
- net +12V: track 0.00 -> 86.3 mm
- net Net-(Nano1-Pad21): track 0.00 -> 77.8 mm
- net Net-(Nano1-Pad8): track 0.00 -> 65.7 mm
- net Net-(J6-Pad6): track 0.00 -> 45.3 mm
- net Net-(Driver1-Pad9): track 0.00 -> 41.7 mm
- net Net-(Nano1-Pad20): track 0.00 -> 38.6 mm
- net Net-(J6-Pad8): track 0.00 -> 34.7 mm
- net Net-(Driver1-Pad4): track 0.00 -> 30.3 mm
- net Net-(Driver1-Pad5): track 0.00 -> 28.0 mm
- net Net-(J6-Pad7): track 0.00 -> 27.7 mm
- net Net-(Driver1-Pad3): track 0.00 -> 26.6 mm
- net Net-(J6-Pad5): track 0.00 -> 26.3 mm
- net Net-(Driver1-Pad6): track 0.00 -> 25.6 mm
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Other:
- net class Power: trace_width 1 -> 0.7
- board text added: "+"
- board text added: "+12V"
- board text added: "1A"
- board text added: "1B"
- board text added: "2A"
- board text added: "2B"
- board text added: "<- USB"
- board text added: "Ext"
- board text added: "Flash"
- board text added: "Frames"
- board text added: "Leds"
- board text added: "Power"
- board text added: "Speed"
- board text added: "ZOETROPE V1"
- board text removed: "+12v"

Commit message: final revision of PCB V1
Parts:
- moved R2 10.2 mm to (148.6, 78.7), turned to 270 degrees
- moved R3 10.2 mm to (154.9, 88.9), turned to 90 degrees
Connections:
- Nano1 pad 9: GND -> Net-(Nano1-Pad9)
- R3 pad 2: GND -> Net-(Nano1-Pad9)
Routing:
- net Net-(Nano1-Pad9): track 0.00 -> 78.4 mm
- net +5V: track 200.1 -> 188.1 mm, vias 1 -> 2
- net Net-(Q2-Pad1): track 8.89 -> 18.5 mm
- net Net-(Driver1-Pad12): track 8.80 -> 17.7 mm, vias 1 -> 0
- net Net-(Nano1-Pad8): track 65.7 -> 70.3 mm
- net +12V: track 86.3 -> 89.1 mm
- net GND: track 226.7 -> 225.0 mm
- net Net-(J6-Pad6): track 45.3 -> 44.0 mm
- net Net-(Q1-Pad1): track 19.4 -> 18.4 mm
- net Net-(Driver1-Pad9): track 41.7 -> 40.9 mm
Other:
- board text removed: "Flash"
- board text removed: "Frames"
- board text removed: "Speed"
