File: hardware/pcb_kicad/pcb_kicad.kicad_pcb (KiCad board)
At the start: 2 copper layers, 105.4 x 43.2 mm, 24 parts, among them J1 Screw_Terminal_01x02, J2 Screw_Terminal_01x02, J3 Screw_Terminal_01x02, J4 Screw_Terminal_01x02, J5 Screw_Terminal_01x02, J6 Conn_02x05_Counter_Clockwise, Q1 IRLB8721PBF, Q2 IRLB8721PBF, U1 LM7805_TO220

Commit message: pcb V2 wip
Parts:
- J6: value Conn_02x05_Counter_Clockwise -> Conn_02x05_Odd_Even
Connections:
- net /dir renamed /DIR
- net /enable renamed /ENABLE
- net /led1 renamed /LED1
- net /led2 renamed /LED2
- net /step renamed /STEP
- J6 pad 1: Net-(J6-Pad1) -> +5V
- J6 pad 2: Net-(J6-Pad2) -> GND
- J6 pad 3: Net-(J6-Pad3) -> /D2
- J6 pad 4: Net-(J6-Pad4) -> (no net)
- J6 pad 5: Net-(J6-Pad5) -> /D3
- J6 pad 6: Net-(J6-Pad6) -> (no net)
- J6 pad 7: (no net) -> /D7
- J6 pad 9: (no net) -> /D8
- Nano1 pad 10: Net-(J6-Pad3) -> /D7
- Nano1 pad 11: Net-(J6-Pad4) -> /D8
- Nano1 pad 22: Net-(J6-Pad5) -> (no net)
- Nano1 pad 23: Net-(J6-Pad6) -> (no net)
- Nano1 pad 5: Net-(J6-Pad1) -> /D2
- Nano1 pad 6: Net-(J6-Pad2) -> /D3
Routing:
- net Net-(J6-Pad5): track 39.7 -> 0.00 mm
- net GND: track 197.7 -> 234.9 mm
- net /D3: track 0.00 -> 34.4 mm
- net Net-(J6-Pad6): track 27.7 -> 0.00 mm
- net /D7: track 0.00 -> 26.1 mm
- net /D2: track 0.00 -> 24.4 mm
- net /D8: track 0.00 -> 21.3 mm
- net Net-(J6-Pad1): track 20.2 -> 0.00 mm
- net Net-(J6-Pad2): track 18.7 -> 0.00 mm
- net Net-(J6-Pad3): track 15.4 -> 0.00 mm
- net /LED2: track 94.7 -> 106.4 mm, vias 1 -> 0
- net /ENABLE: track 68.4 -> 77.9 mm
- net /MS3: track 75.3 -> 66.0 mm
- net Net-(J6-Pad4): track 7.93 -> 0.00 mm
- net /LED1: track 83.2 -> 77.5 mm
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Other:
- board size 105.4 x 43.2 mm -> 105.4 x 41.9 mm
- board text added: "ZOETROPE V2"
- board text removed: "ZOETROPE V1.1"

Commit message: latest V
Routing:
- net +5V: track 183.9 -> 207.3 mm
- net GND: track 234.9 -> 250.0 mm
- net Net-(Nano1-Pad21): track 81.6 -> 77.8 mm
- net +12V: track 114.6 -> 112.6 mm
- net /D3: track 34.4 -> 33.7 mm
- net /D2: track 24.4 -> 23.9 mm
