File: hardware/pcb_kicad/pcb_kicad.sch (KiCad schematic (older format))
At the start: 26 parts, among them J1 Barrel_Jack, J2 Screw_Terminal_01x02, J3 Screw_Terminal_01x02, J4 Screw_Terminal_01x02, J5 Screw_Terminal_01x02, J6 Conn_01x06_Male, J7 Conn_01x05_Male, Q1 IRLB8721PBF, Q2 IRLB8721PBF

Commit message: best run so far
Parts:
- removed J6: Conn_01x06_Male, Connector_PinHeader_2.54mm:PinHeader_1x06_P2.54mm_Vertical, symbol Connector:Conn_01x06_Male
- removed J7: Conn_01x05_Male, Connector_PinHeader_2.54mm:PinHeader_1x05_P2.54mm_Vertical, symbol Connector:Conn_01x05_Male
- added J6: Conn_02x05_Top_Bottom, Connector_IDC:IDC-Header_2x05_P2.54mm_Vertical, symbol Connector_Generic:Conn_02x05_Top_Bottom
- added U1: LM7805_TO220, Package_TO_SOT_THT:TO-220-3_Vertical, symbol Regulator_Linear:LM7805_TO220
Connections:
- net +12V: now also U1.1 (VI); no longer Nano1.30 (VIN)
- net +5V: now also J6.9 (Pin_9), U1.3 (VO)
- net GND: now also J6.10 (Pin_10), U1.2 (GND); no longer Nano1.10 (D7), Nano1.9 (D6), R3.2
- net at Nano1.11 (D8): now also J6.2 (Pin_2)
- net at Nano1.12 (D9): now also J6.3 (Pin_3)
- net at Nano1.13 (D10): now also J6.4 (Pin_4)
- net at Nano1.22 (A3): now also J6.5 (Pin_5)
- net at Nano1.23 (A4): now also J6.6 (Pin_6)
- net at Nano1.24 (A5): now also J6.7 (Pin_7)
- net at Nano1.25 (A6): now also J6.8 (Pin_8)
- new net: J6.1 (Pin_1), Nano1.10 (D7)
- new net: Nano1.9 (D6), R3.2
- no-connect marks 0 -> 11
Other:
- moved on the sheet: R3
Changed lines of the file:
@@
 	1850 3200 2150 3200
 Wire Wire Line
-	2150 3200 2150 4550
+	2150 3200 2150 4300
 $Comp
 L power:GND #PWR04
 U 1 1 6157E58B
-P 7300 4250
-F 0 "#PWR04" H 7300 4000 50  0001 C CNN
-F 1 "GND" H 7305 4077 50  0000 C CNN
-F 2 "" H 7300 4250 50  0001 C CNN
-F 3 "" H 7300 4250 50  0001 C CNN
-	1    7300 4250
+P 7300 4200
+F 0 "#PWR04" H 7300 3950 50  0001 C CNN
+F 1 "GND" H 7305 4027 50  0000 C CNN
+F 2 "" H 7300 4200 50  0001 C CNN
+F 3 "" H 7300 4200 50  0001 C CNN
+	1    7300 4200
 	1    0    0    -1
 $EndComp
@@
 $EndComp
 $Comp
-L power:+12V #PWR03
-U 1 1 61580843
-P 3150 1450
-F 0 "#PWR03" H 3150 1300 50  0001 C CNN
-F 1 "+12V" H 3165 1623 50  0000 C CNN
-F 2 "" H 3150 1450 50  0001 C CNN
-F 3 "" H 3150 1450 50  0001 C CNN
-	1    3150 1450
-	1    0    0    -1
-$EndComp
-Wire Wire Line
-	3150 2300 3200 2300
-$Comp
 L power:GND #PWR0101
 U 1 1 61585660
@@
 $EndComp
 Wire Wire Line
-	3150 1450 3150 2300
-$Comp
-L MCU_Module:Arduino_Nano_v3.x Nano1
-U 1 1 61571B58
-P 3300 3300
-F 0 "Nano1" H 3300 2211 50  0000 C CNN
-F 1 "Arduino_Nano_v3.x" H 3300 2120 50  0000 C CNN
-F 2 "Module:Arduino_Nano" H 3300 3300 50  0001 C CIN
-F 3 "http://www.mouser.com/pdfdocs/Gravitech_Arduino_Nano3_0.pdf" H 3300 3300 50  0001 C CNN
-	1    3300 3300
-	1    0    0    -1
-$EndComp
-Wire Wire Line
 	3350 4300 3350 5150
 Connection ~ 3350 5150
@@
 Wire Wire Line
 	3350 4300 3400 4300
-$Comp
-L power:+5V #PWR06
-U 1 1 6159371C
-P 3550 1700
-F 0 "#PWR06" H 3550 1550 50  0001 C CNN
-F 1 "+5V" H 3565 1873 50  0000 C CNN
-F 2 "" H 3550 1700 50  0001 C CNN
-F 3 "" H 3550 1700 50  0001 C CNN
-	1    3550 1700
-	1    0    0    -1
-$EndComp
-Wire Wire Line
-	3500 2300 3500 1700
-Wire Wire Line
-	3500 1700 3550 1700
 $Comp
 L power:+5V #PWR09
@@
 L Device:R R3
 U 1 1 615B25FE
-P 5100 5050
-F 0 "R3" V 4893 5050 50  0000 C CNN
-F 1 "220" V 4984 5050 50  0000 C CNN
-F 2 "Resistor_THT:R_Axial_DIN0207_L6.3mm_D2.5mm_P10.16mm_Horizontal" V 5030 5050 50  0001 C CNN
-F 3 "~" H 5100 5050 50  0001 C CNN
-	1    5100 5050
+P 5200 5050
+F 0 "R3" V 4993 5050 50  0000 C CNN
+F 1 "220" V 5084 5050 50  0000 C CNN
+F 2 "Resistor_THT:R_Axial_DIN0207_L6.3mm_D2.5mm_P10.16mm_Horizontal" V 5130 5050 50  0001 C CNN
+F 3 "~" H 5200 5050 50  0001 C CNN
+	1    5200 5050
 	0    1    1    0
 $EndComp
@@
 	4650 4950 4650 6450
 Wire Wire Line
-	5250 5050 5350 5050
-Wire Wire Line
 	5350 5750 5350 5050
 Connection ~ 5350 5050
 Wire Wire Line
-	4200 4550 2700 4550
-Wire Wire Line
-	2700 4550 2700 3200
-Wire Wire Line
-	2700 3200 2800 3200
-Wire Wire Line
-	4950 5050 2600 5050
-Wire Wire Line
-	2600 5050 2600 3300
-Wire Wire Line
 	2600 3300 2800 3300
-Wire Wire Line
-	5650 5500 2500 5500
-Wire Wire Line
-	2500 5500 2500 3400
-Wire Wire Line
-	2500 3400 2800 3400
-Wire Wire Line
-	4950 4750 4950 5050
 Connection ~ 4950 6450
 Wire Wire Line
 	4950 6450 5350 6450
-Connection ~ 4950 5050
-Wire Wire Line
-	4950 5050 4950 6450
-Wire Wire Line
-	5650 5250 5650 5500
 Wire Wire Line
 	5650 6450 5600 6450
-Connection ~ 5650 5500
-Wire Wire Line
-	5650 5500 5650 6450
 Wire Wire Line
 	4950 4350 7750 4350
@@
 	7350 5350 8000 5350
 $Comp
-L Connector:Conn_01x06_Male J6
-U 1 1 6163D794
-P 2600 3700
-F 0 "J6" H 2708 4081 50  0000 C CNN
-F 1 "Conn_01x06_Male" H 2708 3990 50  0000 C CNN
-F 2 "Connector_PinHeader_2.54mm:PinHeader_1x06_P2.54mm_Vertical" H 2600 3700 50  0001 C CNN
-F 3 "~" H 2600 3700 50  0001 C CNN
-	1    2600 3700
-	1    0    0    -1
-$EndComp
-$Comp
-L Connector:Conn_01x05_Male J7
-U 1 1 6163FB69
-P 4000 3800
-F 0 "J7" H 3972 3732 50  0000 R CNN
-F 1 "Conn_01x05_Male" H 3972 3823 50  0000 R CNN
-F 2 "Connector_PinHeader_2.54mm:PinHeader_1x05_P2.54mm_Vertical" H 4000 3800 50  0001 C CNN
-F 3 "~" H 4000 3800 50  0001 C CNN
-	1    4000 3800
-	-1   0    0    1
-$EndComp
-$Comp
 L Mechanical:MountingHole H1
 U 1 1 6164DDB5
@@
 Wire Wire Line
 	7800 3200 7950 3200
+$Comp
+L Regulator_Linear:LM7805_TO220 U1
+U 1 1 615E50B0
+P 1500 4000
+F 0 "U1" H 1500 4242 50  0000 C CNN
+F 1 "LM7805_TO220" H 1500 4151 50  0000 C CNN
+F 2 "Package_TO_SOT_THT:TO-220-3_Vertical" H 1500 4225 50  0001 C CIN
+F 3 "https://www.onsemi.cn/PowerSolutions/document/MC7800-D.PDF" H 1500 3950 50  0001 C CNN
+	1    1500 4000
+	1    0    0    -1
+$EndComp
+$Comp
+L power:+12V #PWR0105
+U 1 1 615F4EE2
+P 1000 3650
+F 0 "#PWR0105" H 1000 3500 50  0001 C CNN
+F 1 "+12V" H 1015 3823 50  0000 C CNN
+F 2 "" H 1000 3650 50  0001 C CNN
+F 3 "" H 1000 3650 50  0001 C CNN
+	1    1000 3650
+	1    0    0    -1
+$EndComp
+Wire Wire Line
+	1000 3650 1000 4000
+Wire Wire Line
+	1000 4000 1200 4000
+Wire Wire Line
+	1500 4300 2150 4300
+Connection ~ 2150 4300
+Wire Wire Line
+	2150 4300 2150 4550
+$Comp
+L MCU_Module:Arduino_Nano_v3.x Nano1
+U 1 1 61571B58
+P 3300 3300
+F 0 "Nano1" H 3300 2211 50  0000 C CNN
+F 1 "Arduino_Nano_v3.x" H 3300 2120 50  0000 C CNN
+F 2 "Module:Arduino_Nano" H 3300 3300 50  0001 C CIN
+F 3 "http://www.mouser.com/pdfdocs/Gravitech_Arduino_Nano3_0.pdf" H 3300 3300 50  0001 C CNN
+	1    3300 3300
+	1    0    0    -1
+$EndComp
+$Comp
+L power:+5V #PWR0106
+U 1 1 616122A8
+P 1900 3650
+F 0 "#PWR0106" H 1900 3500 50  0001 C CNN
+F 1 "+5V" H 1915 3823 50  0000 C CNN
+F 2 "" H 1900 3650 50  0001 C CNN
+F 3 "" H 1900 3650 50  0001 C CNN
+	1    1900 3650
+	1    0    0    -1
+$EndComp
+Wire Wire Line
+	1900 3650 1900 4000
+Wire Wire Line
+	1900 4000 1800 4000
+$Comp
+L power:+5V #PWR0107
+U 1 1 61619272
+P 3500 1650
+F 0 "#PWR0107" H 3500 1500 50  0001 C CNN
+F 1 "+5V" H 3515 1823 50  0000 C CNN
+F 2 "" H 3500 1650 50  0001 C CNN
+F 3 "" H 3500 1650 50  0001 C CNN
+	1    3500 1650
+	1    0    0    -1
+$EndComp
+Wire Wire Line
+	3500 1650 3500 2300
+Wire Wire Line
+	2600 3300 2600 5050
+Wire Wire Line
+	5650 5250 5650 6450
+Wire Wire Line
+	2800 3200 2500 3200
+Wire Wire Line
+	2500 3200 2500 4550
+Wire Wire Line
+	2500 4550 4200 4550
+$Comp
+L power:+5V #PWR010
+U 1 1 616CDADD
+P 3050 6050
+F 0 "#PWR010" H 3050 5900 50  0001 C CNN
+F 1 "+5V" H 3065 6223 50  0000 C CNN
+F 2 "" H 3050 6050 50  0001 C CNN
+F 3 "" H 3050 6050 50  0001 C CNN
+	1    3050 6050
+	-1   0    0    1
+$EndComp
+$Comp
+L power:GND #PWR011
+U 1 1 616D2F37
+P 2850 6300
+F 0 "#PWR011" H 2850 6050 50  0001 C CNN
+F 1 "GND" H 2855 6127 50  0000 C CNN
+F 2 "" H 2850 6300 50  0001 C CNN
+F 3 "" H 2850 6300 50  0001 C CNN
+	1    2850 6300
+	1    0    0    -1
+$EndComp
+$Comp
+L Connector_Generic:Conn_02x05_Top_Bottom J6
+U 1 1 616176B4
+P 2550 5800
+F 0 "J6" H 2600 6217 50  0000 C CNN
+F 1 "Conn_02x05_Top_Bottom" H 2600 6126 50  0000 C CNN
+F 2 "Connector_IDC:IDC-Header_2x05_P2.54mm_Vertical" H 2550 5800 50  0001 C CNN
+F 3 "~" H 2550 5800 50  0001 C CNN
+	1    2550 5800
+	1    0    0    -1
+$EndComp
+Wire Wire Line
+	2850 6300 2850 6000
+Wire Wire Line
+	2800 3400 2450 3400
+Wire Wire Line
+	2450 3400 2450 5400
+Wire Wire Line
+	2450 5400 2350 5400
+Wire Wire Line
+	2350 5400 2350 5600
+Wire Wire Line
+	2800 3500 2800 3550
+Wire Wire Line
+	2800 3550 2400 3550
+Wire Wire Line
+	2400 3550 2400 5350
+Wire Wire Line
+	2400 5350 2250 5350
+Wire Wire Line
+	2250 5350 2250 5700
+Wire Wire Line
+	2250 5700 2350 5700
+Wire Wire Line
+	2800 3600 2350 3600
+Wire Wire Line
+	2350 3600 2350 5250
+Wire Wire Line
+	2350 5250 2100 5250
+Wire Wire Line
+	2100 5250 2100 5800
+Wire Wire Line
+	2100 5800 2350 5800
+Wire Wire Line
+	2800 3700 2300 3700
+Wire Wire Line
+	2300 3700 2300 5150
+Wire Wire Line
+	2300 5150 2000 5150
+Wire Wire Line
+	2000 5150 2000 5900
+Wire Wire Line
+	2000 5900 2350 5900
+NoConn ~ 2800 2800
+NoConn ~ 2800 2700
+NoConn ~ 3800 3100
+NoConn ~ 3800 2800
+NoConn ~ 3800 2700
+NoConn ~ 3400 2300
+NoConn ~ 3200 2300
+NoConn ~ 2800 4000
+NoConn ~ 2800 3900
+NoConn ~ 2800 3800
+NoConn ~ 3800 4000
+Wire Wire Line
+	3050 6050 3050 5900
+Wire Wire Line
+	3050 5900 2850 5900
+Wire Wire Line
+	2350 6000 2350 6600
+Wire Wire Line
+	2350 6600 3950 6600
+Wire Wire Line
+	3950 6600 3950 3600
+Wire Wire Line
+	3950 3600 3800 3600
+Wire Wire Line
+	3800 3700 4000 3700
+Wire Wire Line
+	4000 3700 4000 5600
+Wire Wire Line
+	4000 5600 2850 5600
+Wire Wire Line
+	3800 3800 4050 3800
+Wire Wire Line
+	4050 3800 4050 5700
+Wire Wire Line
+	4050 5700 2850 5700
+Wire Wire Line
+	3800 3900 4100 3900
+Wire Wire Line
+	4100 3900 4100 5800
+Wire Wire Line
+	4100 5800 2850 5800
+Wire Wire Line
+	4950 4750 4950 6450
+Wire Wire Line
+	2600 5050 5050 5050
 $EndSCHEMATC

Commit message: v2 to be checked
Parts:
- removed J1: Barrel_Jack, TerminalBlock:TerminalBlock_bornier-2_P5.08mm, symbol Connector:Barrel_Jack
- removed JP1, JP2, JP3: SolderJumper_3_Bridged12, Jumper:SolderJumper-3_P1.3mm_Bridged12_Pad1.0x1.5mm_NumberLabels, symbol Jumper:SolderJumper_3_Bridged12
- added D1: 1N4004, Diode_THT:D_DO-41_SOD81_P10.16mm_Horizontal, symbol Diode:1N4004
- added J1: Screw_Terminal_01x02, TerminalBlock:TerminalBlock_bornier-2_P5.08mm, symbol Connector:Screw_Terminal_01x02
- added R5: 100K, Resistor_THT:R_Axial_DIN0207_L6.3mm_D2.5mm_P10.16mm_Horizontal, symbol Device:R
Connections:
- net +12V: now also D1.1 (K)
- net +5V: now also R5.1
- net GND: now also J1.1 (Pin_1)
- net MS1: now reaches Nano1.14 (D11)
- net MS1: now also Driver1.10 (MS1)
- net MS2: now reaches Nano1.15 (D12)
- net MS2: now also Driver1.11 (MS2)
- net MS3: now reaches Nano1.16 (D13)
- net MS3: now also Driver1.12 (MS3)
- net at Driver1.9 (~ENABLE), Nano1.7 (D4): now also R5.2
- new net: D1.2 (A), J1.2 (Pin_2)
- no-connect marks 11 -> 8
Changed lines of the file:
@@
-$EndComp
-$Comp
-L Connector:Barrel_Jack J1
-U 1 1 6157563F
-P 1550 3100
-F 0 "J1" H 1607 3425 50  0000 C CNN
-F 1 "Barrel_Jack" H 1607 3334 50  0000 C CNN
-F 2 "TerminalBlock:TerminalBlock_bornier-2_P5.08mm" H 1600 3060 50  0001 C CNN
-F 3 "~" H 1600 3060 50  0001 C CNN
-	1    1550 3100
-	1    0    0    -1
 $EndComp
 $Comp
@@
 $EndComp
 Wire Wire Line
-	1850 3000 2250 3000
-Wire Wire Line
-	2250 3000 2250 2300
-Wire Wire Line
-	1850 3200 2150 3200
-Wire Wire Line
 	2150 3200 2150 4300
 $Comp
@@
 Wire Wire Line
 	2450 1900 6300 1900
-Wire Wire Line
-	6300 1900 6300 2900
 Wire Wire Line
 	6300 2900 6900 2900
@@
 	9350 4200 7500 4200
 Connection ~ 7500 4200
-$Comp
-L Jumper:SolderJumper_3_Bridged12 JP1
-U 1 1 615C72FF
-P 6000 3300
-F 0 "JP1" V 6046 3368 50  0000 L CNN
-F 1 "SolderJumper_3_Bridged12" V 5955 3368 50  0000 L CNN
-F 2 "Jumper:SolderJumper-3_P1.3mm_Bridged12_Pad1.0x1.5mm_NumberLabels" H 6000 3300 50  0001 C CNN
-F 3 "~" H 6000 3300 50  0001 C CNN
-	1    6000 3300
-	0    -1   -1   0
-$EndComp
-$Comp
-L Jumper:SolderJumper_3_Bridged12 JP2
-U 1 1 615C93FC
-P 6350 3400
-F 0 "JP2" V 6396 3468 50  0000 L CNN
-F 1 "SolderJumper_3_Bridged12" V 6305 3468 50  0000 L CNN
-F 2 "Jumper:SolderJumper-3_P1.3mm_Bridged12_Pad1.0x1.5mm_NumberLabels" H 6350 3400 50  0001 C CNN
-F 3 "~" H 6350 3400 50  0001 C CNN
-	1    6350 3400
-	0    -1   -1   0
-$EndComp
-$Comp
-L Jumper:SolderJumper_3_Bridged12 JP3
-U 1 1 615CF697
-P 6550 3550
-F 0 "JP3" V 6596 3618 50  0000 L CNN
-F 1 "SolderJumper_3_Bridged12" V 6505 3618 50  0000 L CNN
-F 2 "Jumper:SolderJumper-3_P1.3mm_Bridged12_Pad1.0x1.5mm_NumberLabels" H 6550 3550 50  0001 C CNN
-F 3 "~" H 6550 3550 50  0001 C CNN
-	1    6550 3550
-	0    -1   -1   0
-$EndComp
-Wire Wire Line
-	6750 3500 6900 3500
-Wire Wire Line
-	6500 3400 6900 3400
-Wire Wire Line
-	6000 3500 6000 4200
-Wire Wire Line
-	6000 4200 6350 4200
-Wire Wire Line
-	6350 3600 6350 4200
-Connection ~ 6350 4200
-$Comp
-L power:+5V #PWR0104
-U 1 1 615E6AAC
-P 6150 3100
-F 0 "#PWR0104" H 6150 2950 50  0001 C CNN
-F 1 "+5V" H 6165 3273 50  0000 C CNN
-F 2 "" H 6150 3100 50  0001 C CNN
-F 3 "" H 6150 3100 50  0001 C CNN
-	1    6150 3100
-	1    0    0    -1
-$EndComp
-Wire Wire Line
-	6150 3100 6000 3100
-Wire Wire Line
-	6150 3100 6350 3100
-Wire Wire Line
-	6350 3100 6350 3200
-Connection ~ 6150 3100
-Wire Wire Line
-	6700 3550 6750 3550
-Wire Wire Line
-	6750 3550 6750 3500
-Wire Wire Line
-	6150 3300 6900 3300
-Wire Wire Line
-	6550 3350 6550 3200
-Wire Wire Line
-	6550 3200 6350 3200
-Connection ~ 6350 3200
-Wire Wire Line
-	6350 4200 6550 4200
-Wire Wire Line
-	6550 3750 6550 4200
-Connection ~ 6550 4200
-Wire Wire Line
-	6550 4200 7300 4200
 Wire Wire Line
 	7350 5350 8000 5350
@@
 NoConn ~ 3400 2300
 NoConn ~ 3200 2300
-NoConn ~ 2800 4000
-NoConn ~ 2800 3900
-NoConn ~ 2800 3800
 NoConn ~ 3800 4000
 Wire Wire Line
@@
 Wire Wire Line
 	2600 5050 5050 5050
+Wire Wire Line
+	1650 3200 1650 3150
+Wire Wire Line
+	1650 3200 2150 3200
+$Comp
+L Diode:1N4004 D1
+U 1 1 6175F83B
+P 1950 3050
+F 0 "D1" H 1950 2834 50  0000 C CNN
+F 1 "1N4004" H 1950 2925 50  0000 C CNN
+F 2 "Diode_THT:D_DO-41_SOD81_P10.16mm_Horizontal" H 1950 2875 50  0001 C CNN
+F 3 "http://www.vishay.com/docs/88503/1n4001.pdf" H 1950 3050 50  0001 C CNN
+	1    1950 3050
+	-1   0    0    1
+$EndComp
+$Comp
+L Connector:Screw_Terminal_01x02 J1
+U 1 1 6174A9AD
+P 1450 3150
+F 0 "J1" H 1368 2825 50  0000 C CNN
+F 1 "Screw_Terminal_01x02" H 1368 2916 50  0000 C CNN
+F 2 "TerminalBlock:TerminalBlock_bornier-2_P5.08mm" H 1450 3150 50  0001 C CNN
+F 3 "~" H 1450 3150 50  0001 C CNN
+	1    1450 3150
+	-1   0    0    1
+$EndComp
+Wire Wire Line
+	1650 3050 1800 3050
+Wire Wire Line
+	2100 3050 2250 3050
+Wire Wire Line
+	2250 3050 2250 2300
+$Comp
+L Device:R R5
+U 1 1 6177F9D0
+P 6300 1500
+F 0 "R5" H 6370 1546 50  0000 L CNN
+F 1 "100K" H 6370 1455 50  0000 L CNN
+F 2 "Resistor_THT:R_Axial_DIN0207_L6.3mm_D2.5mm_P10.16mm_Horizontal" V 6230 1500 50  0001 C CNN
+F 3 "~" H 6300 1500 50  0001 C CNN
+	1    6300 1500
+	1    0    0    -1
+$EndComp
+Wire Wire Line
+	6300 1650 6300 1900
+Connection ~ 6300 1900
+Wire Wire Line
+	6300 1900 6300 2900
+$Comp
+L power:+5V #PWR03
+U 1 1 61787A07
+P 6300 1150
+F 0 "#PWR03" H 6300 1000 50  0001 C CNN
+F 1 "+5V" H 6315 1323 50  0000 C CNN
+F 2 "" H 6300 1150 50  0001 C CNN
+F 3 "" H 6300 1150 50  0001 C CNN
+	1    6300 1150
+	1    0    0    -1
+$EndComp
+Wire Wire Line
+	6300 1150 6300 1350
+Text Label 6600 3300 2    50   ~ 0
+MS1
+Text Label 6600 3400 2    50   ~ 0
+MS2
+Text Label 6600 3500 2    50   ~ 0
+MS3
+Wire Wire Line
+	6600 3300 6900 3300
+Wire Wire Line
+	6600 3400 6900 3400
+Wire Wire Line
+	6600 3500 6900 3500
+Text Label 2750 3800 2    50   ~ 0
+MS1
+Text Label 2750 3900 2    50   ~ 0
+MS2
+Text Label 2750 4000 2    50   ~ 0
+MS3
+Wire Wire Line
+	2750 3800 2800 3800
+Wire Wire Line
+	2750 3900 2800 3900
+Wire Wire Line
+	2750 4000 2800 4000
 $EndSCHEMATC
